Commit message: Formatted W200 attachment URDF

File: clearpath_platform_description/urdf/w200/attachments/arm_mount.urdf.xacro (robot description, xacro)
@@ -1,6 +1,6 @@
 <?xml version="1.0"?>
 <robot xmlns:xacro="http://ros.org/wiki/xacro">
-  <xacro:macro name="w200_arm_mount">
-    <link name="arm_mount_link">
+  <xacro:macro name="arm_mount" params="name:=arm_mount model:=default parent_link:=default_mount *origin">
+    <link name="${name}_link">
       <visual>
         <origin xyz="0 0 0" rpy="0 0 0"/>
@@ -22,4 +22,9 @@
       </inertial>
     </link>
+    <joint name="${name}_link_joint" type="fixed">
+      <xacro:insert_block name="origin"/>
+      <parent link="${parent_link}"/>
+      <child link="${name}_link" />
+    </joint>
   </xacro:macro>
 </robot>

File: clearpath_platform_description/urdf/w200/attachments/generator.urdf.xacro (robot description, xacro)
@@ -1,6 +1,6 @@
 <?xml version="1.0"?>
 <robot xmlns:xacro="http://www.ros.org/wiki/xacro">
-  <xacro:macro name="w200_generator">
-    <link name="generator_link">
+  <xacro:macro name="generator" params="name:=generator model:=default parent_link:=mid_mount *origin">
+    <link name="${name}_link">
       <visual>
         <origin xyz="0 0 0" rpy="0 0 0"/>
@@ -22,4 +22,9 @@
       </inertial>
     </link>
+    <joint name="${name}_link_joint" type="fixed">
+      <xacro:insert_block name="origin"/>
+      <parent link="${parent_link}"/>
+      <child link="${name}_link"/>
+    </joint>
   </xacro:macro>
 </robot>

Commit message: Arm Mount at base

File: clearpath_platform_description/urdf/w200/attachments/arm_mount.urdf.xacro (robot description, xacro)
@@ -4,5 +4,5 @@
     <link name="${name}_link">
       <visual>
-        <origin xyz="0 0 0" rpy="0 0 0"/>
+        <origin xyz="0 0 0.02" rpy="0 0 0"/>
         <geometry>
           <mesh filename="package://clearpath_platform_description/meshes/w200/arm-mount-plate.stl" />
@@ -11,5 +11,5 @@
       </visual>
       <collision>
-        <origin xyz="0 0 0" rpy="0 0 0"/>
+        <origin xyz="0 0 0.02" rpy="0 0 0"/>
         <geometry>
           <mesh filename="package://clearpath_platform_description/meshes/w200/arm-mount-plate.stl" />

File: clearpath_platform_description/urdf/w200/attachments/bulkhead.urdf.xacro (robot description, xacro)
@@ -36,5 +36,5 @@
     <xacro:if value="${model == 'arm_mount'}">
       <xacro:arm_mount parent_link="${name}_front_mount_link">
-        <origin xyz="0.0 0.0 0.02" rpy="0.0 0.0 0.0"/>
+        <origin xyz="0.0 0.0 0.0" rpy="0.0 0.0 0.0"/>
       </xacro:arm_mount>
     </xacro:if>
