Commit message: Added  to materials

File: clearpath_mounts_description/urdf/disk.urdf.xacro (robot description, xacro)
@@ -4,5 +4,5 @@
     <link name="${name}_link">
       <visual>
-        <material name="dark_grey"/>
+        <material name="clearpath_dark_grey"/>
         <geometry>
           <mesh filename="package://clearpath_mounts_description/meshes/disk.stl" />

File: clearpath_mounts_description/urdf/pacs/bracket.urdf.xacro (robot description, xacro)
@@ -89,5 +89,5 @@
     <link name="${name}_link">
       <visual>
-          <material name="dark_grey"/>
+          <material name="clearpath_dark_grey"/>
           <geometry>
             <mesh filename="${mesh}" />

File: clearpath_mounts_description/urdf/pacs/riser.urdf.xacro (robot description, xacro)
@@ -49,5 +49,5 @@
           </xacro:unless>
         </geometry>
-        <material name="dark_grey" />
+        <material name="clearpath_dark_grey" />
         <origin xyz="${-(rows / 2) * spacing + spacing / 2} ${-(columns / 2) * spacing + spacing / 2} ${thickness / 2}" rpy="0 0 0" />
       </visual>
@@ -57,5 +57,5 @@
           <box size="0.11 0.59 ${thickness}" />
         </geometry>
-        <material name="dark_grey" />
+        <material name="clearpath_dark_grey" />
       </collision>
     </link>

File: clearpath_mounts_description/urdf/pacs/riser_leg.urdf.xacro (robot description, xacro)
@@ -33,5 +33,5 @@
           <box size="0.04 0.02 ${height}" />
         </geometry>
-        <material name="dark_grey" />
+        <material name="clearpath_dark_grey" />
       </visual>
       <collision>
@@ -40,5 +40,5 @@
           <box size="0.04 0.02 ${height}" />
         </geometry>
-        <material name="dark_grey" />
+        <material name="clearpath_dark_grey" />
       </collision>
     </link>

File: clearpath_mounts_description/urdf/post.urdf.xacro (robot description, xacro)
@@ -31,5 +31,5 @@
       <xacro:if value="${post_model == 'single'}">
         <visual>
-          <material name="light_grey" />
+          <material name="clearpath_light_grey" />
           <origin xyz="0 0 ${height/2}" />
           <geometry>
@@ -48,5 +48,5 @@
         <!-- Left -->
         <visual>
-          <material name="light_grey" />
+          <material name="clearpath_light_grey" />
           <origin xyz="0 ${spacing/2} ${height/2}" />
           <geometry>
@@ -62,5 +62,5 @@
         <!-- Right -->
         <visual>
-          <material name="light_grey" />
+          <material name="clearpath_light_grey" />
           <origin xyz="0 ${-spacing/2} ${height/2}" />
           <geometry>
@@ -79,5 +79,5 @@
         <!-- Front Left -->
         <visual>
-          <material name="light_grey" />
+          <material name="clearpath_light_grey" />
           <origin xyz="${spacing/2} ${spacing/2} ${height/2}" />
           <geometry>
@@ -93,5 +93,5 @@
         <!-- Front Right -->
         <visual>
-          <material name="light_grey" />
+          <material name="clearpath_light_grey" />
           <origin xyz="${spacing/2} ${-spacing/2} ${height/2}" />
           <geometry>
@@ -107,5 +107,5 @@
         <!-- Rear Left -->
         <visual>
-          <material name="light_grey" />
+          <material name="clearpath_light_grey" />
           <origin xyz="${-spacing/2} ${spacing/2} ${height/2}" />
           <geometry>
@@ -121,5 +121,5 @@
         <!-- Rear Right -->
         <visual>
-          <material name="light_grey" />
+          <material name="clearpath_light_grey" />
           <origin xyz="${-spacing/2} ${-spacing/2} ${height/2}" />
           <geometry>

File: clearpath_mounts_description/urdf/sick.urdf.xacro (robot description, xacro)
@@ -20,5 +20,5 @@
       <xacro:if value="${model == 'upright'}">
         <visual>
-          <material name="dark_grey" />
+          <material name="clearpath_dark_grey" />
           <geometry>
             <mesh filename="package://clearpath_mounts_description/meshes/sick_upright.stl" />

File: clearpath_platform_description/urdf/a200/attachments/bumper.urdf.xacro (robot description, xacro)
@@ -30,5 +30,5 @@
                         <cylinder radius="0.0095" length="${extension}" />
                     </geometry>
-                    <material name="dark_grey" />
+                    <material name="clearpath_dark_grey" />
                     <origin xyz="${extension / 2} 0 0" rpy="0 ${M_PI/2} 0" />
                 </visual>
@@ -39,5 +39,5 @@
                         <cylinder radius="0.0095" length="${extension}" />
                     </geometry>
-                    <material name="dark_grey" />
+                    <material name="clearpath_dark_grey" />
                     <origin xyz="${extension / 2} 0 0" rpy="0 ${M_PI/2} 0" />
                 </visual>

File: clearpath_platform_description/urdf/a200/attachments/top_plate.urdf.xacro (robot description, xacro)
@@ -98,6 +98,5 @@
         <link name="${name}_link">
           <visual>
-            <origin xyz="0.0483 0 0"/>
-            <material name="dark_grey" />
+            <material name="clearpath_dark_grey" />
             <geometry>
               <mesh filename="package://clearpath_platform_description/meshes/a200/attachments/pacs_top_plate.stl" />
@@ -105,6 +104,6 @@
           </visual>
           <collision>
-            <material name="dark_grey" />
-            <origin xyz="0.0483 0 0.003175" rpy="0 0 0"/>
+            <material name="clearpath_dark_grey" />
+            <origin xyz="0 0 0.00317500531673" rpy="0 0 0"/>
             <geometry>
               <box size="0.67 0.59 0.00635"/>

File: clearpath_platform_description/urdf/common.urdf.xacro (robot description, xacro)
@@ -23,16 +23,16 @@
 -->
 <robot xmlns:xacro="http://ros.org/wiki/xacro">
-    <material name="dark_grey"><color rgba="0.2 0.2 0.2 1.0" /></material>
-    <material name="medium_grey"><color rgba="0.6 0.6 0.6 1.0" /></material>
-    <material name="light_grey"><color rgba="0.8 0.8 0.8 1.0" /></material>
-    <material name="yellow"><color rgba="0.8 0.8 0.0 1.0" /></material>
-    <material name="black"><color rgba="0.15 0.15 0.15 1.0" /></material>
-    <material name="white"><color rgba="1.0 1.0 1.0 1.0" /></material>
-    <material name="red"><color rgba="1.0 0.0 0.0 1.0" /></material>
-    <material name="aluminum">
+    <material name="clearpath_dark_grey"><color rgba="0.2 0.2 0.2 1.0" /></material>
+    <material name="clearpath_medium_grey"><color rgba="0.6 0.6 0.6 1.0" /></material>
+    <material name="clearpath_light_grey"><color rgba="0.8 0.8 0.8 1.0" /></material>
+    <material name="clearpath_yellow"><color rgba="0.8 0.8 0.0 1.0" /></material>
+    <material name="clearpath_black"><color rgba="0.15 0.15 0.15 1.0" /></material>
+    <material name="clearpath_white"><color rgba="1.0 1.0 1.0 1.0" /></material>
+    <material name="clearpath_red"><color rgba="1.0 0.0 0.0 1.0" /></material>
+    <material name="clearpath_aluminum">
       <color rgba="0.5 0.5 0.5 1"/>
     </material>
-    <material name="plastic">
-      <color rgba="0.1 0.1 0.1 1"/>
+    <material name="clearpath_plastic">
+      <color rgba="0.1 0.1 0.1   1"/>
     </material>
     <!--

File: clearpath_platform_description/urdf/j100/accessories/bridge_plate.urdf.xacro (robot description, xacro)
@@ -19,5 +19,5 @@
           <mesh filename="package://clearpath_platform_description/meshes/j100/bridge_plate.stl"/>
         </geometry>
-        <material name="dark_grey" />
+        <material name="clearpath_dark_grey" />
       </visual>
     </link>

File: clearpath_platform_description/urdf/j100/accessories/camera_mount.urdf.xacro (robot description, xacro)
@@ -7,5 +7,5 @@
           <mesh filename="package://clearpath_platform_description/meshes/j100/camera_bracket.stl" scale="0.001 0.001 0.001" />
         </geometry>
-        <material name="dark_grey" />
+        <material name="clearpath_dark_grey" />
       </visual>
     </link>
@@ -16,5 +16,5 @@
           <mesh filename="package://clearpath_platform_description/meshes/j100/camera_beam.stl" scale="0.001 0.001 0.001" />
         </geometry>
-        <material name="dark_grey" />
+        <material name="clearpath_dark_grey" />
       </visual>
     </link>

File: clearpath_platform_description/urdf/j100/accessories/hdl32_mount.urdf.xacro (robot description, xacro)
@@ -9,5 +9,5 @@
           </geometry>
           <origin xyz="0 0 0" rpy="0 0 0" />
-          <material name="black" />
+          <material name="clearpath_black" />
         </visual>
         <collision>

File: clearpath_platform_description/urdf/j100/accessories/sick_lms1xx_mount.urdf.xacro (robot description, xacro)
@@ -41,5 +41,5 @@
           <mesh filename="package://clearpath_platform_description/meshes/j100/sick_lms1xx_bracket.stl" />
         </geometry>
-        <material name="dark_grey" />
+        <material name="clearpath_dark_grey" />
       </visual>
     </link>

File: clearpath_platform_description/urdf/j100/accessories/standoffs.urdf.xacro (robot description, xacro)
@@ -9,5 +9,5 @@
           <cylinder radius="0.004" length="${length}" />
         </geometry>
-        <material name="light_grey" />
+        <material name="clearpath_light_grey" />
       </visual>
     </link>

File: clearpath_platform_description/urdf/j100/accessories/stereo_camera_mount.urdf.xacro (robot description, xacro)
@@ -8,5 +8,5 @@
           <mesh filename="package://clearpath_platform_description/meshes/j100/stereo_camera_bracket.stl" />
         </geometry>
-        <material name="dark_grey" />
+        <material name="clearpath_dark_grey" />
       </visual>
     </link>
@@ -17,5 +17,5 @@
           <mesh filename="package://clearpath_platform_description/meshes/j100/stereo_camera_beam.stl" />
         </geometry>
-        <material name="dark_grey" />
+        <material name="clearpath_dark_grey" />
       </visual>
     </link>

File: clearpath_platform_description/urdf/j100/accessories/vlp16_mount.urdf.xacro (robot description, xacro)
@@ -8,5 +8,5 @@
           <box size="0.1 0.1 0.002" />
         </geometry>
-        <material name="black" />
+        <material name="clearpath_black" />
         <origin xyz="0 0 -0.001" rpy="0 0 0" />
       </visual>
@@ -17,5 +17,5 @@
           <cylinder length="${height}" radius="0.003" />
         </geometry>
-        <material name="white">
+        <material name="clearpath_white">
           <color rgba="1 1 1 1" />
         </material>
@@ -28,5 +28,5 @@
           <cylinder length="${height}" radius="0.003" />
         </geometry>
-        <material name="white">
+        <material name="clearpath_white">
           <color rgba="1 1 1 1" />
         </material>
@@ -39,5 +39,5 @@
           <cylinder length="${height}" radius="0.003" />
         </geometry>
-        <material name="white">
+        <material name="clearpath_white">
           <color rgba="1 1 1 1" />
         </material>
@@ -50,5 +50,5 @@
           <cylinder length="${height}" radius="0.003" />
         </geometry>
-        <material name="white">
+        <material name="clearpath_white">
           <color rgba="1 1 1 1" />
         </material>

File: clearpath_platform_description/urdf/j100/attachments/front_fender.urdf.xacro (robot description, xacro)
@@ -1,7 +1,7 @@
 <?xml version="1.0"?>
 <robot xmlns:xacro="http://ros.org/wiki/xacro">
-  <xacro:macro name="fender" params="name model parent_link:=base_link *origin">
+  <xacro:macro name="front_fender" params="model *origin">
     <!-- Spawn fender link -->
-    <link name="${name}_link">
+    <link name="front_fender_link">
       <visual>
         <geometry>
@@ -17,16 +17,16 @@
     </link>
     <xacro:if value="${model == 'sensor'}">
-      <link name="${name}_mount"/>
-      <joint name="${name}_mount_joint" type="fixed">
+      <link name="front_fender_mount"/>
+      <joint name="front_fender_mount_joint" type="fixed">
         <origin xyz="0.25629 0 0.07455" rpy="${pi} 0 0" />
-        <parent link="${name}_link" />
-        <child link="${name}_mount" />
+        <parent link="front_fender_link" />
+        <child link="front_fender_mount" />
       </joint>
     </xacro:if>
     <!-- Attach fender -->
-    <joint name="${name}_joint" type="fixed">
-      <xacro:insert_block name="origin"/>
-      <parent link="${parent_link}" />
-      <child link="${name}_link" />
+    <joint name="front_fender_joint" type="fixed">
+      <origin xyz="0 0 0" rpy="0 0 0"/>
+      <parent link="base_link" />
+      <child link="front_fender_link" />
     </joint>
   </xacro:macro>

File: clearpath_platform_description/urdf/j100/attachments/top_plate.urdf.xacro (robot description, xacro)
@@ -9,5 +9,5 @@
               <mesh filename="package://clearpath_platform_description/meshes/j100/attachments/ark_enclosure.stl"/>
             </geometry>
-            <material name="dark_grey" />
+            <material name="clearpath_dark_grey" />
           </visual>
         </link>

File: clearpath_platform_description/urdf/j100/j100.urdf.xacro (robot description, xacro)
@@ -72,5 +72,5 @@
           <mesh filename="package://clearpath_platform_description/meshes/j100/j100_base.stl"/>
         </geometry>
-        <material name="dark_grey" />
+        <material name="clearpath_dark_grey" />
       </visual>
       <collision>
@@ -118,5 +118,5 @@
         </geometry>
         <origin xyz="0 0 0.008" />
-        <material name="black" />
+        <material name="clearpath_black" />
       </visual>
     </link>

File: clearpath_platform_description/urdf/j100/wheel.urdf.xacro (robot description, xacro)
@@ -8,5 +8,5 @@
           <mesh filename="package://clearpath_platform_description/meshes/j100/j100_wheel.stl"/>
         </geometry>
-        <material name="black" />
+        <material name="clearpath_black" />
       </visual>
       <collision>
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