Commit message: Attachment URDF match changes

File: clearpath_platform_description/urdf/a200/attachments/bumper.urdf.xacro (robot description, xacro)
@@ -1,9 +1,5 @@
 <?xml version="1.0"?>
 <robot xmlns:xacro="http://ros.org/wiki/xacro">
-    <xacro:macro name="bumper" params="name extension:=0 *origin">
-        <xacro:property name="parent_link" value="front_bumper_mount" />
-        <xacro:if value="${'rear' in name}" >
-            <xacro:property name="parent_link" value="rear_bumper_mount" />
-        </xacro:if>
+    <xacro:macro name="bumper" params="name model:='default' parent_link:='front_bumper_mount' extension:=0 *origin">
         <!-- Spawn bumper link -->
         <link name="${name}_link">

File: clearpath_platform_description/urdf/a200/attachments/sensor_arch.urdf.xacro (robot description, xacro)
@@ -1,8 +1,8 @@
 <?xml version="1.0"?>
 <robot xmlns:xacro="http://ros.org/wiki/xacro" name="510_mm_sensor_arch">
-  <xacro:macro name="structure" params="parent_link model:=sensor_arch_510 *origin">
+  <xacro:macro name="sensor_arch" params="name parent_link model:=sensor_arch_510 *origin">
     <xacro:if value="${model == 'sensor_arch_510'}">
       <!-- Spawn the sensor arch link -->
-      <link name="sensor_arch_link">
+      <link name="${name}_link">
         <visual>
           <origin xyz="0 0 0.51" rpy="0 0 0"/>
@@ -18,20 +18,20 @@
         </collision>
       </link>
-      <link name="sensor_arch_mount"/>
+      <link name="${name}_mount"/>
       <!-- Attach the sensor arch to the top plate -->
-      <joint name="sensor_arch_joint" type="fixed">
+      <joint name="${name}_joint" type="fixed">
         <xacro:insert_block name="origin"/>
         <parent link="${parent_link}"/>
-        <child link="sensor_arch_link"/>
+        <child link="${name}_link"/>
       </joint>
       <joint name="sensor_arch_mount_joint" type="fixed">
         <origin xyz="0 0 0.51" rpy="0 0 0"/>
-        <parent link="sensor_arch_link"/>
-        <child link="sensor_arch_mount"/>
+        <parent link="${name}_link"/>
+        <child link="${name}_mount"/>
       </joint>
     </xacro:if>
     <xacro:if value="${model == 'sensor_arch_300'}">
       <!-- Spawn the sensor arch link -->
-      <link name="sensor_arch_link">
+      <link name="${name}_link">
         <visual>
           <origin xyz="0 0 0.3" rpy="0 0 0"/>
@@ -47,15 +47,15 @@
         </collision>
       </link>
-      <link name="sensor_arch_mount"/>
+      <link name="${name}_mount"/>
       <!-- Attach the sensor arch to the top plate -->
-      <joint name="sensor_arch_joint" type="fixed">
+      <joint name="${name}_joint" type="fixed">
         <xacro:insert_block name="origin"/>
         <parent link="${parent_link}"/>
-        <child link="sensor_arch_link"/>
+        <child link="${name}_link"/>
       </joint>
-      <joint name="sensor_arch_mount_joint" type="fixed">
+      <joint name="${name}_mount_joint" type="fixed">
         <origin xyz="0 0 0.3" rpy="0 0 0"/>
-        <parent link="sensor_arch_link"/>
-        <child link="sensor_arch_mount"/>
+        <parent link="${name}_link"/>
+        <child link="${name}_mount"/>
       </joint>
     </xacro:if>

File: clearpath_platform_description/urdf/a200/attachments/top_plate.urdf.xacro (robot description, xacro)
@@ -2,8 +2,8 @@
 <robot xmlns:xacro="http://ros.org/wiki/xacro">
     <!-- <xacro:include filename="$(find clearpath_platform_description)/urdf/common.urdf.xacro" /> -->
-    <xacro:macro name="top_plate" params="model:=default *origin">
+    <xacro:macro name="top_plate" params="name model:=default parent_link:=base_link *origin">
         <!-- Spawn the top plate -->
       <xacro:if value="${model == 'large'}">
-        <link name="top_plate_link">
+        <link name="${name}_link">
           <visual>
             <origin xyz="0 0 0" rpy="0 0 0" />
@@ -20,26 +20,26 @@
         </link>
         <!-- Attach top plate -->
-        <joint name="top_plate_joint" type="fixed">
-          <parent link="base_link" />
-          <child link="top_plate_link"/>
+        <joint name="${name}_joint" type="fixed">
+          <parent link="${parent_link}" />
+          <child link="${name}_link"/>
           <origin xyz="0.0812 0 0.225" rpy="0 0 0"/>
         </joint>
         <!-- Top plate front link -->
-        <joint name="top_plate_front_joint" type="fixed">
-          <parent link="top_plate_link" />
-          <child link="top_plate_front_link"/>
+        <joint name="${name}_front_joint" type="fixed">
+          <parent link="${name}_link" />
+          <child link="${name}_front_link"/>
           <origin xyz="0.4125 0 0.00672" rpy="0 0 0"/>
         </joint>
         <!-- Top plate rear link-->
-        <joint name="top_plate_rear_joint" type="fixed">
-          <parent link="top_plate_link" />
-          <child link="top_plate_rear_link"/>
+        <joint name="${name}_rear_joint" type="fixed">
+          <parent link="${name}_link" />
+          <child link="${name}_rear_link"/>
           <origin xyz="-0.4125 0 0.00672" rpy="0 0 0"/>
         </joint>
-        <link name="top_plate_front_link"/>
-        <link name="top_plate_rear_link"/>
+        <link name="${name}_front_link"/>
+        <link name="${name}_rear_link"/>
       </xacro:if>
       <xacro:if value="${model == 'default'}">
-        <link name="top_plate_link">
+        <link name="${name}_link">
           <visual>
             <origin xyz="0 0 0" rpy="0 0 0" />
@@ -56,19 +56,19 @@
         </link>
         <!-- Attach top plate -->
-        <joint name="top_plate_joint" type="fixed">
-          <parent link="base_link" />
-          <child link="top_plate_link"/>
+        <joint name="${name}_joint" type="fixed">
+          <parent link="${parent_link}" />
+          <child link="${name}_link"/>
           <origin xyz="0.0812 0 0.245" rpy="0 0 0"/>
         </joint>
         <!-- Top plate front link -->
-        <joint name="top_plate_front_joint" type="fixed">
-          <parent link="top_plate_link" />
-          <child link="top_plate_front_link"/>
+        <joint name="${name}_front_joint" type="fixed">
+          <parent link="${name}_link" />
+          <child link="${name}_front_link"/>
           <origin xyz="0.36367 0 0.00639" rpy="0 0 0"/>
         </joint>
         <!-- Top plate rear link-->
-        <joint name="top_plate_rear_joint" type="fixed">
-          <parent link="top_plate_link" />
-          <child link="top_plate_rear_link"/>
+        <joint name="${name}_rear_joint" type="fixed">
+          <parent link="${name}_link" />
+          <child link="${name}_rear_link"/>
           <origin xyz="-0.36633 0 0.00639" rpy="0 0 0"/>
         </joint>
@@ -87,9 +87,9 @@
           <child link="user_rail_link" />
         </joint>
-        <link name="top_plate_front_link"/>
-        <link name="top_plate_rear_link"/>
+        <link name="${name}_front_link"/>
+        <link name="${name}_rear_link"/>
       </xacro:if>
       <xacro:if value="${model == 'pacs'}">
-        <link name="top_plate_link">
+        <link name="${name}_link">
           <visual>
             <material name="dark_grey" />
@@ -107,13 +107,13 @@
         </link>
         <!-- Attach PACS top plate -->
-        <joint name="top_plate_joint" type="fixed">
-          <child link="top_plate_link"/>
-          <parent link="base_link"/>
+        <joint name="${name}_joint" type="fixed">
+          <child link="${name}_link"/>
+          <parent link="${parent_link}"/>
           <origin xyz="0.048299998045 0 0.227500006557" rpy="0 0 0"/>
         </joint>
         <!-- Generate PACS mounts -->
         <xacro:full_mounts
-          name="top_plate"
-          parent_link="top_plate_link"
+          name="${name}"
+          parent_link="${name}_link"
           column="a"
           row="1"
@@ -124,6 +124,6 @@
           z="0.00635" />
         <xacro:full_mounts
-          name="top_plate"
-          parent_link="top_plate_link"
+          name="${name}"
+          parent_link="${name}_link"
           column="a"
           row="3"
@@ -134,6 +134,6 @@
           z="0.00635" />
         <xacro:full_mounts
-          name="top_plate"
-          parent_link="top_plate_link"
+          name="${name}"
+          parent_link="${name}_link"
           column="g"
           row="3"
@@ -144,6 +144,6 @@
           z="0.00635" />
         <xacro:full_mounts
-          name="top_plate"
-          parent_link="top_plate_link"
+          name="${name}"
+          parent_link="${name}_link"
           column="a"
           row="7"

File: clearpath_platform_description/urdf/j100/attachments/fender.urdf.xacro (robot description, xacro)
@@ -1,7 +1,7 @@
 <?xml version="1.0"?>
 <robot xmlns:xacro="http://ros.org/wiki/xacro">
-  <xacro:macro name="rear_fender" params="model *origin">
+  <xacro:macro name="fender" params="name model parent_link:=base_link *origin">
     <!-- Spawn fender link -->
-    <link name="rear_fender_link">
+    <link name="${name}_link">
       <visual>
         <geometry>
@@ -17,16 +17,16 @@
     </link>
     <xacro:if value="${model == 'sensor'}">
-      <link name="rear_fender_mount"/>
-      <joint name="rear_fender_mount_joint" type="fixed">
+      <link name="${name}_mount"/>
+      <joint name="${name}_mount_joint" type="fixed">
         <origin xyz="0.25629 0 0.07455" rpy="${pi} 0 0" />
-        <parent link="rear_fender_link" />
-        <child link="rear_fender_mount" />
+        <parent link="${name}_link" />
+        <child link="${name}_mount" />
       </joint>
     </xacro:if>
     <!-- Attach fender -->
-    <joint name="rear_fender_joint" type="fixed">
-      <origin xyz="0 0 0" rpy="0 0 ${pi}"/>
-      <parent link="base_link" />
-      <child link="rear_fender_link" />
+    <joint name="${name}_joint" type="fixed">
+      <xacro:insert_block name="origin"/>
+      <parent link="${parent_link}" />
+      <child link="${name}_link" />
     </joint>
   </xacro:macro>

File: clearpath_platform_description/urdf/j100/attachments/top_plate.urdf.xacro (robot description, xacro)
@@ -1,7 +1,7 @@
 <?xml version="1.0"?>
 <robot xmlns:xacro="http://ros.org/wiki/xacro">
-    <xacro:macro name="top_plate" params="model:=default">
+    <xacro:macro name="top_plate" params="name:=ark_enclosure model:=default parent_link:=mid_mount *origin">
       <xacro:if value="${model == 'ark_enclosure'}">
-         <link name="ark_enclosure_link">
+         <link name="${name}_link">
           <visual>
             <origin xyz="0 0 0" rpy="0 0 0"/>
@@ -12,7 +12,8 @@
           </visual>
         </link>
-        <joint name="ark_enclosure_joint" type="fixed">
-          <parent link="mid_mount" />
-          <child link="ark_enclosure_link" />
+        <joint name="${name}_joint" type="fixed">
+          <parent link="${parent_link}" />
+          <child link="${name}_link" />
+          <xacro:insert_block name="origin"/>
         </joint>
       </xacro:if>

Commit message: Origin to bumper

File: clearpath_platform_description/urdf/a200/attachments/bumper.urdf.xacro (robot description, xacro)
@@ -11,8 +11,14 @@
         </link>
         <xacro:unless value="${extension > 0}">
+            <link name="${name}_base_link"/>
+            <joint name="${name}_base_joint" type="fixed">
+                <xacro:insert_block name="origin"/>
+                <parent link="${parent_link}"/>
+                <child link="${name}_base_link"/>
+            </joint>
             <!-- Attach bumper -->
             <joint name="${name}_joint" type="fixed">
                 <origin xyz="0.075 0 0" rpy="0 0 0" />
-                <parent link="${parent_link}" />
+                <parent link="${name}_base_link" />
                 <child link="${name}_link" />
             </joint>
@@ -37,18 +43,24 @@
                 </visual>
             </link>
+            <link name="${name}_base_link"/>
             <link name="${name}_extension_mount"/>
+            <joint name="${name}_base_joint" type="fixed">
+                <xacro:insert_block name="origin"/>
+                <parent link="${parent_link}"/>
+                <child link="${name}_base_link"/>
+            </joint>
             <joint name="${name}_extension_joint_1" type="fixed">
                 <origin xyz="0 0.1084 0" rpy="0 0 0" />
-                <parent link="${parent_link}" />
+                <parent link="${name}_base_link" />
                 <child link="${name}_extension_link_1" />
             </joint>
             <joint name="${name}_extension_joint_2" type="fixed">
                 <origin xyz="0 -0.1084 0" rpy="0 0 0" />
-                <parent link="${parent_link}" />
+                <parent link="${name}_base_link" />
                 <child link="${name}_extension_link_2" />
             </joint>
             <joint name="${name}_extension_mount_joint" type="fixed">
                 <origin xyz="${extension} 0 0" rpy="0 0 0" />
-                <parent link="${parent_link}" />
+                <parent link="${name}_base_link" />
                 <child link="${name}_extension_mount" />
             </joint>
