Commit message: Mounts re-numbering

File: clearpath_platform_description/urdf/a200/attachments/top_plate.urdf.xacro (robot description, xacro)
@@ -26,15 +26,15 @@
         </joint>
         <!-- Top plate front link -->
-        <link name="${name}_front_link"/>
+        <link name="${name}_front_mount"/>
         <joint name="${name}_front_joint" type="fixed">
           <parent link="${name}_link" />
-          <child link="${name}_front_link"/>
+          <child link="${name}_front_mount"/>
           <origin xyz="0.4125 0 0.00672" rpy="0 0 0"/>
         </joint>
         <!-- Top plate rear link-->
-        <link name="${name}_rear_link"/>
+        <link name="${name}_rear_mount"/>
         <joint name="${name}_rear_joint" type="fixed">
           <parent link="${name}_link" />
-          <child link="${name}_rear_link"/>
+          <child link="${name}_rear_mount"/>
           <origin xyz="-0.4125 0 0.00672" rpy="0 0 0"/>
         </joint>
@@ -79,15 +79,15 @@
         </joint>
         <!-- Top plate front link -->
-        <link name="${name}_front_link"/>
+        <link name="${name}_front_mount"/>
         <joint name="${name}_front_joint" type="fixed">
           <parent link="${name}_link" />
-          <child link="${name}_front_link"/>
+          <child link="${name}_front_mount"/>
           <origin xyz="0.36367 0 0.00639" rpy="0 0 0"/>
         </joint>
         <!-- Top plate rear link-->
-        <link name="${name}_rear_link"/>
+        <link name="${name}_rear_mount"/>
         <joint name="${name}_rear_joint" type="fixed">
           <parent link="${name}_link" />
-          <child link="${name}_rear_link"/>
+          <child link="${name}_rear_mount"/>
           <origin xyz="-0.36633 0 0.00639" rpy="0 0 0"/>
         </joint>

File: clearpath_platform_description/urdf/j100/j100.urdf.xacro (robot description, xacro)
@@ -139,14 +139,14 @@
       <origin xyz="0 0 ${chassis_height}" />
     </joint>
-    <link name="rear_mount"></link>
-    <joint name="rear_mount_joint" type="fixed">
+    <link name="rear_0_mount"></link>
+    <joint name="rear_0_mount_joint" type="fixed">
       <parent link="default_mount" />
-      <child link="rear_mount" />
+      <child link="rear_0_mount" />
       <origin xyz="${-mount_spacing} 0 0" />
     </joint>
-    <link name="front_mount"></link>
-    <joint name="front_mount_joint" type="fixed">
+    <link name="front_0_mount"></link>
+    <joint name="front_0_mount_joint" type="fixed">
       <parent link="default_mount" />
-      <child link="front_mount" />
+      <child link="front_0_mount" />
       <origin xyz="${mount_spacing} 0 0" />
     </joint>
