Commit message: Changed sensor arch parent

File: clearpath_platform_description/urdf/a200/attachments/sensor_arch.urdf.xacro (robot description, xacro)
@@ -1,5 +1,5 @@
 <?xml version="1.0"?>
 <robot xmlns:xacro="http://ros.org/wiki/xacro" name="510_mm_sensor_arch">
-  <xacro:macro name="sensor_arch" params="name parent_link model:=sensor_arch_510 *origin">
+  <xacro:macro name="sensor_arch" params="name parent_link:=mid_mount model:=sensor_arch_510 *origin">
     <xacro:if value="${model == 'sensor_arch_510'}">
       <!-- Spawn the sensor arch link -->

Commit message: Changed default parent to default_mount

File: clearpath_platform_description/urdf/a200/attachments/sensor_arch.urdf.xacro (robot description, xacro)
@@ -1,5 +1,5 @@
 <?xml version="1.0"?>
 <robot xmlns:xacro="http://ros.org/wiki/xacro" name="sensor_arch">
-  <xacro:macro name="sensor_arch" params="name parent_link:=mid_mount model:=sensor_arch_510 *origin">
+  <xacro:macro name="sensor_arch" params="name parent_link:=default_mount model:=sensor_arch_510 *origin">
     <xacro:if value="${model == 'sensor_arch_510'}">
       <!-- Spawn the sensor arch link -->

File: clearpath_platform_description/urdf/a200/attachments/top_plate.urdf.xacro (robot description, xacro)
@@ -1,5 +1,5 @@
 <?xml version="1.0"?>
 <robot xmlns:xacro="http://ros.org/wiki/xacro">
-    <xacro:macro name="top_plate" params="name model:=default parent_link:=mid_mount *origin">
+    <xacro:macro name="top_plate" params="name model:=default parent_link:=default_mount *origin">
       <!-- Large Model -->
       <xacro:if value="${model == 'large'}">

File: clearpath_platform_description/urdf/j100/attachments/top_plate.urdf.xacro (robot description, xacro)
@@ -1,5 +1,5 @@
 <?xml version="1.0"?>
 <robot xmlns:xacro="http://ros.org/wiki/xacro">
-    <xacro:macro name="top_plate" params="name:=ark_enclosure model:=default parent_link:=mid_mount *origin">
+    <xacro:macro name="top_plate" params="name:=ark_enclosure model:=default parent_link:=default_mount *origin">
       <xacro:if value="${model == 'ark_enclosure'}">
          <link name="${name}_link">

File: clearpath_platform_description/urdf/w200/attachments/bulkhead.urdf.xacro (robot description, xacro)
@@ -1,5 +1,5 @@
 <?xml version="1.0"?>
 <robot xmlns:xacro="http://www.ros.org/wiki/xacro">
-  <xacro:macro name="bulkhead" params="name:=bulkhead model:=default parent_link:=mid_mount *origin">
+  <xacro:macro name="bulkhead" params="name:=bulkhead model:=default parent_link:=default_mount *origin">
     <xacro:include filename="$(find clearpath_platform_description)/urdf/w200/attachments/arm_mount.urdf.xacro"/>
     <link name="${name}_link">

File: clearpath_platform_description/urdf/w200/attachments/generator.urdf.xacro (robot description, xacro)
@@ -1,5 +1,5 @@
 <?xml version="1.0"?>
 <robot xmlns:xacro="http://www.ros.org/wiki/xacro">
-  <xacro:macro name="generator" params="name:=generator model:=default parent_link:=mid_mount *origin">
+  <xacro:macro name="generator" params="name:=generator model:=default parent_link:=default_mount *origin">
     <link name="${name}_link">
       <visual>
