Commit message: Changed top_chassis_link to default_mount

File: clearpath_platform_description/urdf/w200/w200.urdf.xacro (robot description, xacro)
@@ -314,9 +314,9 @@
       </collision>
     </link>
-    <link name="top_chassis_link"></link>
-    <joint name="top_link_joint" type="fixed">
+    <link name="default_mount"></link>
+    <joint name="default_mount_joint" type="fixed">
       <origin xyz="0 0 0.27218" rpy="0 0 0" />
       <parent link="chassis_link"/>
-      <child link="top_chassis_link" />
+      <child link="default_mount" />
     </joint>
     <!-- This link is purely to complete the visual look -->

Commit message: Set color appropriately

File: clearpath_platform_description/urdf/w200/w200.urdf.xacro (robot description, xacro)
@@ -189,11 +189,4 @@
         <origin xyz="0 0 0" rpy="0 0 ${side*PI/2}"/>
         <geometry>
-          <mesh filename="package://clearpath_platform_description/meshes/w200/rocker.stl" />
-        </geometry>
-        <material name="black"><color rgba="0.15 0.15 0.15 1.0" /></material>
-      </visual>
-      <visual>
-        <origin xyz="0 0 0" rpy="0 0 ${side*PI/2}"/>
-        <geometry>
           <mesh filename="package://clearpath_platform_description/meshes/w200/fenders.stl" />
         </geometry>
@@ -208,4 +201,11 @@
         </geometry>
       </collision>
+      <visual>
+        <origin xyz="0 0 0" rpy="0 0 ${side*PI/2}"/>
+        <geometry>
+          <mesh filename="package://clearpath_platform_description/meshes/w200/rocker.stl" />
+        </geometry>
+        <material name="black"><color rgba="0.15 0.15 0.15 1.0" /></material>
+      </visual>
     </link>
     <joint name="${prefix}_diff_unit_joint" type="revolute">
