Commit message: Moved gazebo controller to common

File: clearpath_platform_description/urdf/a200/a200.urdf.xacro (robot description, xacro)
@@ -1,5 +1,4 @@
 <?xml version="1.0"?>
 <robot xmlns:xacro="http://ros.org/wiki/xacro">
-  <xacro:arg name="gazebo_controllers" default="$(find clearpath_control)/config/a200/control.yaml" />
   <xacro:arg name="namespace" default="" />
   <xacro:arg name="is_sim" default="false" />
@@ -130,35 +129,4 @@
       <child link="rear_bumper_mount" />
     </joint>
-    <!-- Default mount -->
-    <link name="default_mount"/>
-    <joint name="default_mount_joint" type="fixed">
-      <child link="default_mount"/>
-      <parent link="base_link"/>
-      <origin xyz="0.0 0.0 0.224"/>
-    </joint>
-    <xacro:if value="$(arg is_sim)">
-      <gazebo>
-        <plugin filename="libign_ros2_control-system.so" name="ign_ros2_control::IgnitionROS2ControlPlugin">
-          <parameters>$(arg gazebo_controllers)</parameters>
-          <ros>
-            <remapping>~/odom:=platform/odom</remapping>
-            <remapping>~/cmd_vel_unstamped:=platform/cmd_vel_unstamped</remapping>
-            <remapping>/tf:=tf</remapping>
-            <remapping>/tf_static:=tf_static</remapping>
-            <remapping>/diagnostics:=diagnostics</remapping>
-            <remapping>joint_states:=platform/joint_states</remapping>
-            <namespace>$(arg namespace)</namespace>
-          </ros>
-        </plugin>
-      </gazebo>
-      <gazebo>
-        <plugin filename="libignition-gazebo-pose-publisher-system.so" name="ignition::gazebo::systems::PosePublisher">
-          <publish_link_pose>true</publish_link_pose>
-          <publish_nested_model_pose>true</publish_nested_model_pose>
-          <use_pose_vector_msg>true</use_pose_vector_msg>
-          <update_frequency>50</update_frequency>
-        </plugin>
-      </gazebo>
-    </xacro:if>
     <ros2_control name="a200_hardware" type="system">
       <hardware>

File: clearpath_platform_description/urdf/j100/j100.urdf.xacro (robot description, xacro)
@@ -5,5 +5,4 @@
   <xacro:arg name="is_sim" default="false" />
   <xacro:arg name="prefix" default="" />
-  <xacro:arg name="gazebo_controllers" default="$(find clearpath_control)/config/j100/control.yaml" />
   <xacro:arg name="namespace" default="" />
   <xacro:property name="PI" value="3.1415926535897931" />
@@ -151,28 +150,4 @@
       <origin xyz="${mount_spacing} 0 0" />
     </joint>
-    <xacro:if value="$(arg is_sim)">
-      <gazebo>
-        <plugin filename="libign_ros2_control-system.so" name="ign_ros2_control::IgnitionROS2ControlPlugin">
-          <parameters>$(arg gazebo_controllers)</parameters>
-          <ros>
-            <remapping>~/odom:=platform/odom</remapping>
-            <remapping>~/cmd_vel_unstamped:=platform/cmd_vel_unstamped</remapping>
-            <remapping>/tf:=tf</remapping>
-            <remapping>/tf_static:=tf_static</remapping>
-            <remapping>/diagnostics:=diagnostics</remapping>
-            <remapping>joint_states:=platform/joint_states</remapping>
-            <namespace>$(arg namespace)</namespace>
-          </ros>
-        </plugin>
-      </gazebo>
-      <gazebo>
-        <plugin filename="libignition-gazebo-pose-publisher-system.so" name="ignition::gazebo::systems::PosePublisher">
-          <publish_link_pose>true</publish_link_pose>
-          <publish_nested_model_pose>true</publish_nested_model_pose>
-          <use_pose_vector_msg>true</use_pose_vector_msg>
-          <update_frequency>50</update_frequency>
-        </plugin>
-      </gazebo>
-    </xacro:if>
     <!-- ROS2 controls -->
     <ros2_control name="j100_hardware" type="system">

Commit message: Added mid_mount

File: clearpath_platform_description/urdf/a200/a200.urdf.xacro (robot description, xacro)
@@ -129,4 +129,11 @@
       <parent link="base_link" />
       <child link="rear_bumper_mount" />
+    </joint>
+    <!-- Mid mount -->
+    <link name="mid_mount"/>
+    <joint name="mid_mount_joint" type="fixed">
+      <child link="mid_mount"/>
+      <parent link="base_link"/>
+      <origin xyz="0.0 0.0 0.224"/>
     </joint>
     <xacro:if value="$(arg is_sim)">

File: clearpath_platform_description/urdf/a200/attachments/top_plate.urdf.xacro (robot description, xacro)
@@ -1,11 +1,11 @@
 <?xml version="1.0"?>
 <robot xmlns:xacro="http://ros.org/wiki/xacro">
-    <!-- <xacro:include filename="$(find clearpath_platform_description)/urdf/common.urdf.xacro" /> -->
-    <xacro:macro name="top_plate" params="name model:=default parent_link:=base_link *origin">
-        <!-- Spawn the top plate -->
+    <xacro:macro name="top_plate" params="name model:=default parent_link:=mid_mount *origin">
+      <!-- Large Model -->
       <xacro:if value="${model == 'large'}">
+        <!-- Spawn top plate -->
         <link name="${name}_link">
           <visual>
-            <origin xyz="0 0 0" rpy="0 0 0" />
+            <origin xyz="0.0812 0 0" rpy="0 0 0" />
             <geometry>
               <mesh filename="package://clearpath_platform_description/meshes/a200/attachments/large_top_plate.dae" />
@@ -13,5 +13,5 @@
           </visual>
           <collision>
-            <origin xyz="0 0 0" rpy="0 0 0"/>
+            <origin xyz="0.0812 0 0" rpy="0 0 0"/>
             <geometry>
               <mesh filename="package://clearpath_platform_description/meshes/a200/attachments/large_top_plate_collision.stl" />
@@ -23,7 +23,8 @@
           <parent link="${parent_link}" />
           <child link="${name}_link"/>
-          <origin xyz="0.0812 0 0.225" rpy="0 0 0"/>
+          <xacro:insert_block name="origin"/>
         </joint>
         <!-- Top plate front link -->
+        <link name="${name}_front_link"/>
         <joint name="${name}_front_joint" type="fixed">
           <parent link="${name}_link" />
@@ -32,4 +33,5 @@
         </joint>
         <!-- Top plate rear link-->
+        <link name="${name}_rear_link"/>
         <joint name="${name}_rear_joint" type="fixed">
           <parent link="${name}_link" />
@@ -37,11 +39,26 @@
           <origin xyz="-0.4125 0 0.00672" rpy="0 0 0"/>
         </joint>
-        <link name="${name}_front_link"/>
-        <link name="${name}_rear_link"/>
       </xacro:if>
+      <!-- Default Model -->
       <xacro:if value="${model == 'default'}">
+        <!-- Spawn user rails -->
+        <link name="${name}_user_rail_link">
+          <visual>
+            <origin xyz="0.272 0 0.019"/>
+            <geometry>
+              <mesh filename="package://clearpath_platform_description/meshes/a200/attachments/user_rail.dae" />
+            </geometry>
+          </visual>
+        </link>
+        <!-- Attach user rails to base link -->
+        <joint name="${name}_user_rail_joint" type="fixed">
+          <xacro:insert_block name="origin"/>
+          <parent link="${parent_link}" />
+          <child link="${name}_user_rail_link" />
+        </joint>
+        <!-- Spawn top plate -->
         <link name="${name}_link">
           <visual>
-            <origin xyz="0 0 0" rpy="0 0 0" />
+            <origin xyz="0.0812 0 0" rpy="0 0 0" />
             <geometry>
               <mesh filename="package://clearpath_platform_description/meshes/a200/attachments/top_plate.dae" />
@@ -49,5 +66,5 @@
           </visual>
           <collision>
-            <origin xyz="0 0 0" rpy="0 0 0"/>
+            <origin xyz="0.0812 0 0" rpy="0 0 0"/>
             <geometry>
               <mesh filename="package://clearpath_platform_description/meshes/a200/attachments/top_plate.stl" />
@@ -57,9 +74,10 @@
         <!-- Attach top plate -->
         <joint name="${name}_joint" type="fixed">
-          <parent link="${parent_link}" />
+          <parent link="${name}_user_rail_link" />
           <child link="${name}_link"/>
-          <origin xyz="0.0812 0 0.245" rpy="0 0 0"/>
+          <origin xyz="0 0 0.021" rpy="0 0 0"/>
         </joint>
         <!-- Top plate front link -->
+        <link name="${name}_front_link"/>
         <joint name="${name}_front_joint" type="fixed">
           <parent link="${name}_link" />
@@ -68,4 +86,5 @@
         </joint>
         <!-- Top plate rear link-->
+        <link name="${name}_rear_link"/>
         <joint name="${name}_rear_joint" type="fixed">
           <parent link="${name}_link" />
@@ -73,24 +92,11 @@
           <origin xyz="-0.36633 0 0.00639" rpy="0 0 0"/>
         </joint>
-        <!-- Spawn user rails -->
-        <link name="user_rail_link">
-          <visual>
-            <geometry>
-              <mesh filename="package://clearpath_platform_description/meshes/a200/attachments/user_rail.dae" />
-            </geometry>
-          </visual>
-        </link>
-        <!-- Attach user rails to base link -->
-        <joint name="user_rail" type="fixed">
-          <origin xyz="0.272 0 0.245" rpy="0 0 0" />
-          <parent link="base_link" />
-          <child link="user_rail_link" />
-        </joint>
-        <link name="${name}_front_link"/>
-        <link name="${name}_rear_link"/>
       </xacro:if>
+      <!-- PACS Model -->
       <xacro:if value="${model == 'pacs'}">
+        <!-- Spawn top plate -->
         <link name="${name}_link">
           <visual>
+            <origin xyz="0.0483 0 0"/>
             <material name="dark_grey" />
             <geometry>
@@ -100,7 +106,7 @@
           <collision>
             <material name="dark_grey" />
-            <origin xyz="0 0 0.00317500531673" rpy="0 0 0"/>
+            <origin xyz="0.0483 0 0.003175" rpy="0 0 0"/>
             <geometry>
-              <box size="0.670000076294 0.590000033379 0.00635001063347"/>
+              <box size="0.67 0.59 0.00635"/>
             </geometry>
           </collision>
@@ -110,5 +116,5 @@
           <child link="${name}_link"/>
           <parent link="${parent_link}"/>
-          <origin xyz="0.048299998045 0 0.227500006557" rpy="0 0 0"/>
+          <xacro:insert_block name="origin"/>
         </joint>
         <!-- Generate PACS mounts -->

Commit message: Changed mid_mount to default_mount

File: clearpath_platform_description/urdf/a200/a200.urdf.xacro (robot description, xacro)
@@ -130,8 +130,8 @@
       <child link="rear_bumper_mount" />
     </joint>
-    <!-- Mid mount -->
-    <link name="mid_mount"/>
-    <joint name="mid_mount_joint" type="fixed">
-      <child link="mid_mount"/>
+    <!-- Default mount -->
+    <link name="default_mount"/>
+    <joint name="default_mount_joint" type="fixed">
+      <child link="default_mount"/>
       <parent link="base_link"/>
       <origin xyz="0.0 0.0 0.224"/>

File: clearpath_platform_description/urdf/j100/j100.urdf.xacro (robot description, xacro)
@@ -133,13 +133,13 @@
       </sensor>
     </gazebo>
-    <link name="mid_mount"></link>
-    <joint name="mid_mount_joint" type="fixed">
+    <link name="default_mount"></link>
+    <joint name="default_mount_joint" type="fixed">
       <parent link="chassis_link" />
-      <child link="mid_mount" />
+      <child link="default_mount" />
       <origin xyz="0 0 ${chassis_height}" />
     </joint>
     <link name="rear_mount"></link>
     <joint name="rear_mount_joint" type="fixed">
-      <parent link="mid_mount" />
+      <parent link="default_mount" />
       <child link="rear_mount" />
       <origin xyz="${-mount_spacing} 0 0" />
@@ -147,5 +147,5 @@
     <link name="front_mount"></link>
     <joint name="front_mount_joint" type="fixed">
-      <parent link="mid_mount" />
+      <parent link="default_mount" />
       <child link="front_mount" />
       <origin xyz="${mount_spacing} 0 0" />

Commit message: Updated gazebo simulation

File: clearpath_platform_description/urdf/a200/a200.urdf.xacro (robot description, xacro)
@@ -4,4 +4,5 @@
   <xacro:arg name="is_sim" default="false" />
   <xacro:arg name="serial_port" default="/dev/clearpath/prolific" />
+  <xacro:arg name="gazebo_controllers" default="$(find clearpath_control)/config/a200/control.yaml"/>
   <!-- Included URDF/XACRO Files -->
   <xacro:include filename="$(find clearpath_platform_description)/urdf/a200/wheel.urdf.xacro" />
@@ -129,4 +130,14 @@
       <child link="rear_bumper_mount" />
     </joint>
+    <!-- Gazebo Controller -->
+    <xacro:include filename="$(find clearpath_platform_description)/urdf/generic/gazebo.urdf.xacro"/>
+    <joint name="default_mount_joint" type="fixed">
+      <child link="default_mount"/>
+      <parent link="base_link"/>
+      <origin xyz="0.0 0.0 0.224"/>
+    </joint>
+    <!-- Gazebo Controller -->
+    <xacro:include filename="$(find clearpath_platform_description)/urdf/generic/gazebo.urdf.xacro"/>
+    <!-- ROS2 controls -->
     <ros2_control name="a200_hardware" type="system">
       <hardware>

File: clearpath_platform_description/urdf/w200/w200.urdf.xacro (robot description, xacro)
@@ -4,4 +4,5 @@
   <xacro:arg name="namespace" default="" />
   <xacro:arg name="is_sim" default="false" />
+  <xacro:arg name="gazebo_controllers" default="$(find clearpath_control)/config/w200/control.yaml"/>
   <xacro:property name="PI" value="3.1415926535897931"/>
   <xacro:property name="wheel_radius" value="0.3" />
@@ -86,6 +87,6 @@
       <mu1>0.5</mu1>
       <mu2>0.5</mu2>
-      <kp value="10000000.0" />
-      <kd value="1.0" />
+      <!-- <kp value="10000000.0" /> -->
+      <!-- <kd value="1.0" /> -->
       <fdir1 value="1 0 0" />
       <material>Gazebo/DarkGrey</material>
@@ -216,5 +217,5 @@
       </visual>
     </link>
-    <joint name="${prefix}_diff_unit_joint" type="revolute">
+    <joint name="${prefix}_diff_unit_joint" type="fixed">
       <limit upper="0.4" lower="-0.4" effort="100" velocity="1"/>
       <parent link="chassis_link"/>
@@ -356,34 +357,26 @@
       <origin xyz="-0.5826 0 0.24979" rpy="0 0 0" />
     </joint>
-    <link name="imu_link" />
-    <joint name="imu_link_joint" type="fixed">
-      <origin xyz="$(optenv WARTHOG_IMU_XYZ 0 0 0)" rpy="$(optenv WARTHOG_IMU_RPY 0 0 0)" />
-      <parent link="chassis_link"/>
-      <child link="imu_link" />
-    </joint>
-     <xacro:if value="$(arg is_sim)">
-      <gazebo>
-        <plugin filename="libign_ros2_control-system.so" name="ign_ros2_control::IgnitionROS2ControlPlugin">
-          <parameters>$(arg gazebo_controllers)</parameters>
-          <ros>
-            <remapping>~/odom:=platform/odom</remapping>
-            <remapping>~/cmd_vel_unstamped:=platform/cmd_vel_unstamped</remapping>
-            <remapping>/tf:=tf</remapping>
-            <remapping>/tf_static:=tf_static</remapping>
-            <remapping>/diagnostics:=diagnostics</remapping>
-            <remapping>joint_states:=platform/joint_states</remapping>
-            <namespace>$(arg namespace)</namespace>
-          </ros>
-        </plugin>
-      </gazebo>
-      <gazebo>
-        <plugin filename="libignition-gazebo-pose-publisher-system.so" name="ignition::gazebo::systems::PosePublisher">
-          <publish_link_pose>true</publish_link_pose>
-          <publish_nested_model_pose>true</publish_nested_model_pose>
-          <use_pose_vector_msg>true</use_pose_vector_msg>
-          <update_frequency>50</update_frequency>
-        </plugin>
-      </gazebo>
-    </xacro:if>
+    <link name="imu_0_link">
+      <inertial>
+        <mass value="0.001"/>
+        <origin xyz="0 0 0" rpy="0 0 0"/>
+        <inertia ixx="${dummy_inertia}" ixy="0.0" ixz="0.0" iyy="${dummy_inertia}" iyz="0.0" izz="${dummy_inertia}"/>
+      </inertial>
+    </link>
+    <joint name="imu_joint" type="fixed">
+      <parent link="chassis_link" />
+      <child link="imu_0_link" />
+    </joint>
+    <gazebo reference="imu_0_link">
+      <sensor type="imu" name="imu_0">
+        <always_on>true</always_on>
+        <update_rate>50</update_rate>
+        <visualize>true</visualize>
+        <ignition_frame_id>imu_0_link</ignition_frame_id>
+      </sensor>
+    </gazebo>
+    <!-- Gazebo Controller -->
+    <xacro:include filename="$(find clearpath_platform_description)/urdf/generic/gazebo.urdf.xacro"/>
+    <!-- ROS2 controls -->
     <ros2_control name="w200_hardware" type="system">
       <hardware>
@@ -425,4 +418,34 @@
       </joint>
     </ros2_control>
+    <xacro:if value="$(arg is_sim)">
+      <gazebo>
+        <plugin filename="libignition-gazebo-wheel-slip-system.so" name="ignition::gazebo::systems::WheelSlip">
+          <wheel link_name="front_left_wheel_link">
+            <slip_compliance_lateral>1.0</slip_compliance_lateral>
+            <slip_compliance_longitudinal>1.0</slip_compliance_longitudinal>
+            <wheel_normal_force>686</wheel_normal_force>
+            <wheel_radius>${wheel_radius}</wheel_radius>
+          </wheel>
+          <wheel link_name="front_right_wheel_link">
+            <slip_compliance_lateral>1.0</slip_compliance_lateral>
+            <slip_compliance_longitudinal>1.0</slip_compliance_longitudinal>
+            <wheel_normal_force>686</wheel_normal_force>
+            <wheel_radius>${wheel_radius}</wheel_radius>
+          </wheel>
+          <wheel link_name="rear_left_wheel_link">
+            <slip_compliance_lateral>1.0</slip_compliance_lateral>
+            <slip_compliance_longitudinal>1.0</slip_compliance_longitudinal>
+            <wheel_normal_force>686</wheel_normal_force>
+            <wheel_radius>${wheel_radius}</wheel_radius>
+          </wheel>
+          <wheel link_name="rear_right_wheel_link">
+            <slip_compliance_lateral>1.0</slip_compliance_lateral>
+            <slip_compliance_longitudinal>1.0</slip_compliance_longitudinal>
+            <wheel_normal_force>686</wheel_normal_force>
+            <wheel_radius>${wheel_radius}</wheel_radius>
+          </wheel>
+        </plugin>
+      </gazebo>
+    </xacro:if>
   </xacro:macro>
 </robot>
