Commit message: Removed transmission and cleaned up URDF

File: clearpath_platform_description/urdf/j100/j100.urdf.xacro (robot description, xacro)
@@ -81,15 +81,9 @@
       </collision>
       <inertial>
-        <!-- Center of mass -->
         <origin xyz="0.012  0.002 0.067" rpy="0 0 0"/>
         <mass value="16.523"/>
-        <!-- Moments of inertia: ( chassis without wheels ) -->
         <inertia ixx="0.3136" ixy="-0.0008" ixz="0.0164" iyy="0.3922" iyz="-0.0009" izz="0.4485"/>
       </inertial>
     </link>
-    <!-- TODO: Make this internal_imu_link or something, and use a mixed-in xacro
-       to supply the joint between it and imu_link. This is important so that imu_link
-       always points to the "active" IMU. When an upgrade IMU is connected, the
-       internal_imu_link should remain, but imu_link should point to the upgrade one. -->
     <link name="imu_0_link">
       <inertial>
@@ -111,5 +105,4 @@
       </sensor>
     </gazebo>
-    <!-- TODO: Same note as applies to imu_link -->
     <link name="gps_0_link">
       <visual>

File: clearpath_platform_description/urdf/j100/wheel.urdf.xacro (robot description, xacro)
@@ -1,4 +1,4 @@
 <?xml version="1.0"?>
-<robot xmlns:xacro="http://ros.org/wiki/xacro" name="a200_wheel">
+<robot xmlns:xacro="http://ros.org/wiki/xacro" name="j100_wheel">
   <xacro:macro name="j100_wheel" params="prefix *joint_pose">
     <link name="${prefix}_wheel_link">
@@ -35,15 +35,4 @@
       <axis xyz="0 1 0" />
     </joint>
-    <!-- In reality, J100 has only two motors, one per side. However, it's more
-         straightforward for Gazebo to simulate as if there's an actuator per wheel. -->
-    <transmission name="${prefix}_wheel_trans">
-      <type>transmission_interface/SimpleTransmission</type>
-      <joint name="${prefix}_wheel">
-        <hardwareInterface>hardware_interface/VelocityJointInterface</hardwareInterface>
-      </joint>
-      <actuator name="${prefix}_actuator">
-        <mechanicalReduction>1</mechanicalReduction>
-      </actuator>
-    </transmission>
   </xacro:macro>
 </robot>
