Commit message: Removed friction on rear_caster

File: clearpath_platform_description/urdf/dd100/dd100.urdf.xacro (robot description, xacro)
@@ -68,59 +68,5 @@
           <wheel_radius>${wheel_radius}</wheel_radius>
         </wheel>
-        <wheel link_name="rear_caster">
-          <slip_compliance_lateral>1.0</slip_compliance_lateral>
-          <slip_compliance_longitudinal>1.0</slip_compliance_longitudinal>
-          <wheel_normal_force>39.2</wheel_normal_force>
-          <wheel_radius>${wheel_radius}</wheel_radius>
-        </wheel>
       </plugin>
-    </gazebo>
-    <!-- Caster -->
-    <link name="rear_caster">
-      <visual>
-        <origin rpy="0 0 0" xyz="0 0 0"/>
-        <geometry>
-          <sphere radius="0.01"/>
-        </geometry>
-        <material name="clearpath_black"/>
-      </visual>
-      <collision>
-        <geometry>
-          <sphere radius="0.01"/>
-        </geometry>
-        <origin rpy="0 0 0" xyz="0 0 0"/>
-        <surface>
-          <friction>
-            <ode>
-              <mu>0.0</mu>
-              <mu2>0.0</mu2>
-              <slip1>1.0</slip1>
-              <slip2>1.0</slip2>
-            </ode>
-          </friction>
-        </surface>
-      </collision>
-      <inertial>
-        <mass value="0.1" />
-        <origin xyz="0 0 0" />
-        <inertia ixx="0.001" ixy="0.0" ixz="0.0"
-                iyy="0.001" iyz="0.0"
-                izz="0.001" />
-      </inertial>
-    </link>
-    <joint name="rear_caster_joint" type="fixed">
-      <parent link="chassis_link"/>
-      <child link="rear_caster"/>
-      <origin xyz="-0.244 0 -0.00674" rpy="0 0 0"/>
-    </joint>
-    <gazebo reference="rear_caster">
-      <turnGravityOff>false</turnGravityOff>
-      <kp>1000000.0</kp>
-      <kd>100.0</kd>
-      <mu1>0.2</mu1>
-      <mu2>0.2</mu2>
-      <fdir1>1 0 0</fdir1>
-      <minDepth>0.00</minDepth>
-      <implicitSpringDamper>1</implicitSpringDamper>
     </gazebo>
     <!-- Internal IMU -->

Commit message: Added default mount

File: clearpath_platform_description/urdf/dd100/dd100.urdf.xacro (robot description, xacro)
@@ -91,4 +91,5 @@
     </gazebo>
     <!-- Mounting Hard Points -->
+    <link name="default_mount"/>
     <link name="front_2_mount"/>
     <link name="front_1_mount"/>
@@ -97,4 +98,9 @@
     <link name="rear_1_mount"/>
     <link name="rear_0_mount"/>
+    <joint name="default_mount_joint" type="fixed">
+      <origin xyz="0 0 0" rpy="0 0 0"/>
+      <parent link="front_0_mount"/>
+      <child link="default_mount"/>
+    </joint>
     <joint name="front_0_mount_joint" type="fixed">
       <origin xyz="0.040 0 0.064263" rpy="0 0 0" />

Commit message: Re-add caster

File: clearpath_platform_description/urdf/dd100/dd100.urdf.xacro (robot description, xacro)
@@ -70,4 +70,52 @@
       </plugin>
     </gazebo>
+    <!-- Caster -->
+    <link name="rear_caster">
+      <visual>
+        <origin rpy="0 0 0" xyz="0 0 0"/>
+        <geometry>
+          <sphere radius="0.01"/>
+        </geometry>
+        <material name="clearpath_black"/>
+      </visual>
+      <collision>
+        <geometry>
+          <sphere radius="0.01"/>
+        </geometry>
+        <origin rpy="0 0 0" xyz="0 0 0"/>
+        <surface>
+          <friction>
+            <ode>
+              <mu>0.0</mu>
+              <mu2>0.0</mu2>
+              <slip1>1.0</slip1>
+              <slip2>1.0</slip2>
+            </ode>
+          </friction>
+        </surface>
+      </collision>
+      <inertial>
+        <mass value="0.1" />
+        <origin xyz="0 0 0" />
+        <inertia ixx="0.001" ixy="0.0" ixz="0.0"
+                iyy="0.001" iyz="0.0"
+                izz="0.001" />
+      </inertial>
+    </link>
+    <joint name="rear_caster_joint" type="fixed">
+      <parent link="chassis_link"/>
+      <child link="rear_caster"/>
+      <origin xyz="-0.244 0 -0.00674" rpy="0 0 0"/>
+    </joint>
+    <gazebo reference="rear_caster">
+      <turnGravityOff>false</turnGravityOff>
+      <kp>1000000.0</kp>
+      <kd>100.0</kd>
+      <mu1>0.2</mu1>
+      <mu2>0.2</mu2>
+      <fdir1>1 0 0</fdir1>
+      <minDepth>0.00</minDepth>
+      <implicitSpringDamper>1</implicitSpringDamper>
+    </gazebo>
     <!-- Internal IMU -->
     <link name="imu_0_link">
