Commit message: Updated material on flir

File: clearpath_sensors_description/urdf/flir_blackfly.urdf.xacro (robot description, xacro)
@@ -20,5 +20,5 @@
                     <mesh filename="package://clearpath_sensors_description/meshes/flir_blackfly.stl"/>
                 </geometry>
-                <material name="dark_grey" />
+                <material name="clearpath_dark_grey" />
             </visual>
             <collision>
@@ -44,5 +44,5 @@
                 <cylinder radius="0.016" length="0.04"/>
                 </geometry>
-                <material name="dark_grey" />
+                <material name="clearpath_dark_grey" />
             </visual>
             <collision>
